Commit message: 新增 piper 末端控制脚本与 URDF 资源，更新 keyboard的teleop 与 joint limit 模块

File: local_assets/piper.urdf (robot description, URDF)
Before this commit: robot piper_description, 11 links, 10 joints
Links:
- added link gripper; collision sphere radius=0.0001; visual sphere radius=0.005
- link camera: geometry visual mesh filename=meshes/camera.dae
- link camera_mount: geometry visual mesh filename=meshes/camera.dae
Joints:
- added joint link6_to_tcp: type fixed, parent link6, child gripper, origin xyz=0 0 0.15 rpy=0 0 0
